Commit message: Added meshes

File: description/diablo_core.xacro (robot description, xacro)
@@ -29,22 +29,25 @@
       <geometry>
         <mesh
-          filename="package://diablo_viz/meshes/base_link.STL" />
-      </geometry>
-      <material
-        name="">
-        <color
-          rgba="0.752941176470588 0.752941176470588 0.752941176470588 1" />
-      </material>
-    </visual>
-    <collision>
-      <origin
-        xyz="0 0 0"
-        rpy="0 0 0" />
-      <geometry>
-        <mesh
-          filename="package://diablo_viz/meshes/base_link.STL" />
-      </geometry>
-    </collision>
-  </link>
+          filename="package://diablo_bot/meshes/base_link.STL" />
+      </geometry>
+      <material
+        name="">
+        <color
+          rgba="0.752941176470588 0.752941176470588 0.752941176470588 1" />
+      </material>
+    </visual>
+    <collision>
+      <origin
+        xyz="0 0 0"
+        rpy="0 0 0" />
+      <geometry>
+        <mesh
+          filename="package://diablo_bot/meshes/base_link.STL" />
+      </geometry>
+    </collision>
+  </link>
+  <gazebo reference='base_link'>
+    <material>Gazebo/Silver</material>
+  </gazebo>
   <link
     name="l_sho_pitch_Link">
@@ -69,19 +72,19 @@
       <geometry>
         <mesh
-          filename="package://diablo_viz/meshes/l_sho_pitch_Link.STL" />
-      </geometry>
-      <material
-        name="">
-        <color
-          rgba="0.752941176470588 0.752941176470588 0.752941176470588 1" />
-      </material>
-    </visual>
-    <collision>
-      <origin
-        xyz="0 0 0"
-        rpy="0 0 0" />
-      <geometry>
-        <mesh
-          filename="package://diablo_viz/meshes/l_sho_pitch_Link.STL" />
+          filename="package://diablo_bot/meshes/l_sho_pitch_Link.STL" />
+      </geometry>
+      <material
+        name="">
+        <color
+          rgba="0.752941176470588 0.752941176470588 0.752941176470588 1" />
+      </material>
+    </visual>
+    <collision>
+      <origin
+        xyz="0 0 0"
+        rpy="0 0 0" />
+      <geometry>
+        <mesh
+          filename="package://diablo_bot/meshes/l_sho_pitch_Link.STL" />
       </geometry>
     </collision>
@@ -127,19 +130,19 @@
       <geometry>
         <mesh
-          filename="package://diablo_viz/meshes/l_sho_roll_Link.STL" />
-      </geometry>
-      <material
-        name="">
-        <color
-          rgba="0.752941176470588 0.752941176470588 0.752941176470588 1" />
-      </material>
-    </visual>
-    <collision>
-      <origin
-        xyz="0 0 0"
-        rpy="0 0 0" />
-      <geometry>
-        <mesh
-          filename="package://diablo_viz/meshes/l_sho_roll_Link.STL" />
+          filename="package://diablo_bot/meshes/l_sho_roll_Link.STL" />
+      </geometry>
+      <material
+        name="">
+        <color
+          rgba="0.752941176470588 0.752941176470588 0.752941176470588 1" />
+      </material>
+    </visual>
+    <collision>
+      <origin
+        xyz="0 0 0"
+        rpy="0 0 0" />
+      <geometry>
+        <mesh
+          filename="package://diablo_bot/meshes/l_sho_roll_Link.STL" />
       </geometry>
     </collision>
@@ -185,19 +188,19 @@
       <geometry>
         <mesh
-          filename="package://diablo_viz/meshes/l_el_Link.STL" />
-      </geometry>
-      <material
-        name="">
-        <color
-          rgba="0.752941176470588 0.752941176470588 0.752941176470588 1" />
-      </material>
-    </visual>
-    <collision>
-      <origin
-        xyz="0 0 0"
-        rpy="0 0 0" />
-      <geometry>
-        <mesh
-          filename="package://diablo_viz/meshes/l_el_Link.STL" />
+          filename="package://diablo_bot/meshes/l_el_Link.STL" />
+      </geometry>
+      <material
+        name="">
+        <color
+          rgba="0.752941176470588 0.752941176470588 0.752941176470588 1" />
+      </material>
+    </visual>
+    <collision>
+      <origin
+        xyz="0 0 0"
+        rpy="0 0 0" />
+      <geometry>
+        <mesh
+          filename="package://diablo_bot/meshes/l_el_Link.STL" />
       </geometry>
     </collision>
@@ -243,19 +246,19 @@
       <geometry>
         <mesh
-          filename="package://diablo_viz/meshes/l_wrist_Link.STL" />
-      </geometry>
-      <material
-        name="">
-        <color
-          rgba="0.752941176470588 0.752941176470588 0.752941176470588 1" />
-      </material>
-    </visual>
-    <collision>
-      <origin
-        xyz="0 0 0"
-        rpy="0 0 0" />
-      <geometry>
-        <mesh
-          filename="package://diablo_viz/meshes/l_wrist_Link.STL" />
+          filename="package://diablo_bot/meshes/l_wrist_Link.STL" />
+      </geometry>
+      <material
+        name="">
+        <color
+          rgba="0.752941176470588 0.752941176470588 0.752941176470588 1" />
+      </material>
+    </visual>
+    <collision>
+      <origin
+        xyz="0 0 0"
+        rpy="0 0 0" />
+      <geometry>
+        <mesh
+          filename="package://diablo_bot/meshes/l_wrist_Link.STL" />
       </geometry>
     </collision>
@@ -301,19 +304,19 @@
       <geometry>
         <mesh
-          filename="package://diablo_viz/meshes/l_mid_base_Link.STL" />
-      </geometry>
-      <material
-        name="">
-        <color
-          rgba="0.752941176470588 0.752941176470588 0.752941176470588 1" />
-      </material>
-    </visual>
-    <collision>
-      <origin
-        xyz="0 0 0"
-        rpy="0 0 0" />
-      <geometry>
-        <mesh
-          filename="package://diablo_viz/meshes/l_mid_base_Link.STL" />
+          filename="package://diablo_bot/meshes/l_mid_base_Link.STL" />
+      </geometry>
+      <material
+        name="">
+        <color
+          rgba="0.752941176470588 0.752941176470588 0.752941176470588 1" />
+      </material>
+    </visual>
+    <collision>
+      <origin
+        xyz="0 0 0"
+        rpy="0 0 0" />
+      <geometry>
+        <mesh
+          filename="package://diablo_bot/meshes/l_mid_base_Link.STL" />
       </geometry>
     </collision>
@@ -359,19 +362,19 @@
       <geometry>
         <mesh
-          filename="package://diablo_viz/meshes/l_mid_middle_Link.STL" />
-      </geometry>
-      <material
-        name="">
-        <color
-          rgba="0.752941176470588 0.752941176470588 0.752941176470588 1" />
-      </material>
-    </visual>
-    <collision>
-      <origin
-        xyz="0 0 0"
-        rpy="0 0 0" />
-      <geometry>
-        <mesh
-          filename="package://diablo_viz/meshes/l_mid_middle_Link.STL" />
+          filename="package://diablo_bot/meshes/l_mid_middle_Link.STL" />
+      </geometry>
+      <material
+        name="">
+        <color
+          rgba="0.752941176470588 0.752941176470588 0.752941176470588 1" />
+      </material>
+    </visual>
+    <collision>
+      <origin
+        xyz="0 0 0"
+        rpy="0 0 0" />
+      <geometry>
+        <mesh
+          filename="package://diablo_bot/meshes/l_mid_middle_Link.STL" />
       </geometry>
     </collision>
@@ -417,19 +420,19 @@
       <geometry>
         <mesh
-          filename="package://diablo_viz/meshes/l_mid_tip_Link.STL" />
-      </geometry>
-      <material
-        name="">
-        <color
-          rgba="0.752941176470588 0.752941176470588 0.752941176470588 1" />
-      </material>
-    </visual>
-    <collision>
-      <origin
-        xyz="0 0 0"
-        rpy="0 0 0" />
-      <geometry>
-        <mesh
-          filename="package://diablo_viz/meshes/l_mid_tip_Link.STL" />
+          filename="package://diablo_bot/meshes/l_mid_tip_Link.STL" />
+      </geometry>
+      <material
+        name="">
+        <color
+          rgba="0.752941176470588 0.752941176470588 0.752941176470588 1" />
+      </material>
+    </visual>
+    <collision>
+      <origin
+        xyz="0 0 0"
+        rpy="0 0 0" />
+      <geometry>
+        <mesh
+          filename="package://diablo_bot/meshes/l_mid_tip_Link.STL" />
       </geometry>
     </collision>
@@ -475,19 +478,19 @@
       <geometry>
         <mesh
-          filename="package://diablo_viz/meshes/l_thumb_base_Link.STL" />
-      </geometry>
-      <material
-        name="">
-        <color
-          rgba="0.752941176470588 0.752941176470588 0.752941176470588 1" />
-      </material>
-    </visual>
-    <collision>
-      <origin
-        xyz="0 0 0"
-        rpy="0 0 0" />
-      <geometry>
-        <mesh
-          filename="package://diablo_viz/meshes/l_thumb_base_Link.STL" />
+          filename="package://diablo_bot/meshes/l_thumb_base_Link.STL" />
+      </geometry>
+      <material
+        name="">
+        <color
+          rgba="0.752941176470588 0.752941176470588 0.752941176470588 1" />
+      </material>
+    </visual>
+    <collision>
+      <origin
+        xyz="0 0 0"
+        rpy="0 0 0" />
+      <geometry>
+        <mesh
+          filename="package://diablo_bot/meshes/l_thumb_base_Link.STL" />
       </geometry>
     </collision>
@@ -533,19 +536,19 @@
       <geometry>
         <mesh
-          filename="package://diablo_viz/meshes/l_thumb_middle_Link.STL" />
-      </geometry>
-      <material
-        name="">
-        <color
-          rgba="0.752941176470588 0.752941176470588 0.752941176470588 1" />
-      </material>
-    </visual>
-    <collision>
-      <origin
-        xyz="0 0 0"
-        rpy="0 0 0" />
-      <geometry>
-        <mesh
-          filename="package://diablo_viz/meshes/l_thumb_middle_Link.STL" />
+          filename="package://diablo_bot/meshes/l_thumb_middle_Link.STL" />
+      </geometry>
+      <material
+        name="">
+        <color
+          rgba="0.752941176470588 0.752941176470588 0.752941176470588 1" />
+      </material>
+    </visual>
+    <collision>
+      <origin
+        xyz="0 0 0"
+        rpy="0 0 0" />
+      <geometry>
+        <mesh
+          filename="package://diablo_bot/meshes/l_thumb_middle_Link.STL" />
       </geometry>
     </collision>
@@ -591,19 +594,19 @@
       <geometry>
         <mesh
-          filename="package://diablo_viz/meshes/l_thumb_tip_Link.STL" />
-      </geometry>
-      <material
-        name="">
-        <color
-          rgba="0.752941176470588 0.752941176470588 0.752941176470588 1" />
-      </material>
-    </visual>
-    <collision>
-      <origin
-        xyz="0 0 0"
-        rpy="0 0 0" />
-      <geometry>
-        <mesh
-          filename="package://diablo_viz/meshes/l_thumb_tip_Link.STL" />
+          filename="package://diablo_bot/meshes/l_thumb_tip_Link.STL" />
+      </geometry>
+      <material
+        name="">
+        <color
+          rgba="0.752941176470588 0.752941176470588 0.752941176470588 1" />
+      </material>
+    </visual>
+    <collision>
+      <origin
+        xyz="0 0 0"
+        rpy="0 0 0" />
+      <geometry>
+        <mesh
+          filename="package://diablo_bot/meshes/l_thumb_tip_Link.STL" />
       </geometry>
     </collision>
@@ -649,19 +652,19 @@
       <geometry>
         <mesh
-          filename="package://diablo_viz/meshes/l_index_base_Link.STL" />
-      </geometry>
-      <material
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
Commit message: files added

File: description/diablo_core.xacro (robot description, xacro)
@@ -1943,28 +1943,3 @@
     <dynamics damping="0" friction="0"/>
   </joint>
-  <transmission name='trans1'>
-    <type>transmission_interface/SimpleTransmission</type>
-    <joint name="l4">
-      <hardwareInterface>hardware_interface/VelocityJointInterface</hardwareInterface>
-    </joint>
-    <actuator name="motor1">
-      <hardwareInterface>hardware_interface/VelocityJointInterface</hardwareInterface>
-      <mechanicalReduction>1</mechanicalReduction>
-    </actuator>
-  </transmission>
-  <transmission name='trans2'>
-    <type>transmission_interface/SimpleTransmission</type>
-    <joint name="r4">
-      <hardwareInterface>hardware_interface/VelocityJointInterface</hardwareInterface>
-    </joint>
-    <actuator name="motor2">
-      <hardwareInterface>hardware_interface/VelocityJointInterface</hardwareInterface>
-      <mechanicalReduction>1</mechanicalReduction>
-    </actuator>
-  </transmission>
-  <gazebo>
-    <plugin name="gazebo_ros_control" filename="libgazebo_ros_control.so">
-      <robotNamespace>rrbot</robotNamespace>
-    </plugin>
-  </gazebo>
 </robot>

File: description/robot.urdf.xacro (robot description, xacro)
@@ -1,4 +1,12 @@
 <?xml version="1.0"?>
 <robot xmlns:xacro="http://www.ros.org/wiki/xacro"  name="diablo_robot">
+    <xacro:arg name="use_ros2_control" default="true"/>
+    <xacro:arg name="sim_mode" default="false"/>
     <xacro:include filename="diablo_core.xacro" />
+    <xacro:if value="$(arg use_ros2_control)">
+        <xacro:include filename="ros2_control.xacro" />
+    </xacro:if>
+    <xacro:unless value="$(arg use_ros2_control)">
+        <xacro:include filename="gazebo_control.xacro" />
+    </xacro:unless>
 </robot>
