Commit message: New Files Added

File: description/diablo_core.xacro (robot description, xacro)
@@ -29,19 +29,19 @@
       <geometry>
         <mesh
-          filename="package://diablo_bot/meshes/base_link.STL" />
-      </geometry>
-      <material
-        name="">
-        <color
-          rgba="0.752941176470588 0.752941176470588 0.752941176470588 1" />
-      </material>
-    </visual>
-    <collision>
-      <origin
-        xyz="0 0 0"
-        rpy="0 0 0" />
-      <geometry>
-        <mesh
-          filename="package://diablo_bot/meshes/base_link.STL" />
+          filename="$(find diablo_bot)/description/meshes/base_link.STL" />
+      </geometry>
+      <material
+        name="">
+        <color
+          rgba="0.752941176470588 0.752941176470588 0.752941176470588 1" />
+      </material>
+    </visual>
+    <collision>
+      <origin
+        xyz="0 0 0"
+        rpy="0 0 0" />
+      <geometry>
+        <mesh
+          filename="$(find diablo_bot)/description/meshes/base_link.STL" />
       </geometry>
     </collision>
@@ -72,19 +72,19 @@
       <geometry>
         <mesh
-          filename="package://diablo_bot/meshes/l_sho_pitch_Link.STL" />
-      </geometry>
-      <material
-        name="">
-        <color
-          rgba="0.752941176470588 0.752941176470588 0.752941176470588 1" />
-      </material>
-    </visual>
-    <collision>
-      <origin
-        xyz="0 0 0"
-        rpy="0 0 0" />
-      <geometry>
-        <mesh
-          filename="package://diablo_bot/meshes/l_sho_pitch_Link.STL" />
+          filename="$(find diablo_bot)/description/meshes/l_sho_pitch_Link.STL" />
+      </geometry>
+      <material
+        name="">
+        <color
+          rgba="0.752941176470588 0.752941176470588 0.752941176470588 1" />
+      </material>
+    </visual>
+    <collision>
+      <origin
+        xyz="0 0 0"
+        rpy="0 0 0" />
+      <geometry>
+        <mesh
+          filename="$(find diablo_bot)/description/meshes/l_sho_pitch_Link.STL" />
       </geometry>
     </collision>
@@ -130,19 +130,19 @@
       <geometry>
         <mesh
-          filename="package://diablo_bot/meshes/l_sho_roll_Link.STL" />
-      </geometry>
-      <material
-        name="">
-        <color
-          rgba="0.752941176470588 0.752941176470588 0.752941176470588 1" />
-      </material>
-    </visual>
-    <collision>
-      <origin
-        xyz="0 0 0"
-        rpy="0 0 0" />
-      <geometry>
-        <mesh
-          filename="package://diablo_bot/meshes/l_sho_roll_Link.STL" />
+          filename="$(find diablo_bot)/description/meshes/l_sho_roll_Link.STL" />
+      </geometry>
+      <material
+        name="">
+        <color
+          rgba="0.752941176470588 0.752941176470588 0.752941176470588 1" />
+      </material>
+    </visual>
+    <collision>
+      <origin
+        xyz="0 0 0"
+        rpy="0 0 0" />
+      <geometry>
+        <mesh
+          filename="$(find diablo_bot)/description/meshes/l_sho_roll_Link.STL" />
       </geometry>
     </collision>
@@ -188,19 +188,19 @@
       <geometry>
         <mesh
-          filename="package://diablo_bot/meshes/l_el_Link.STL" />
-      </geometry>
-      <material
-        name="">
-        <color
-          rgba="0.752941176470588 0.752941176470588 0.752941176470588 1" />
-      </material>
-    </visual>
-    <collision>
-      <origin
-        xyz="0 0 0"
-        rpy="0 0 0" />
-      <geometry>
-        <mesh
-          filename="package://diablo_bot/meshes/l_el_Link.STL" />
+          filename="$(find diablo_bot)/description/meshes/l_el_Link.STL" />
+      </geometry>
+      <material
+        name="">
+        <color
+          rgba="0.752941176470588 0.752941176470588 0.752941176470588 1" />
+      </material>
+    </visual>
+    <collision>
+      <origin
+        xyz="0 0 0"
+        rpy="0 0 0" />
+      <geometry>
+        <mesh
+          filename="$(find diablo_bot)/description/meshes/l_el_Link.STL" />
       </geometry>
     </collision>
@@ -246,19 +246,19 @@
       <geometry>
         <mesh
-          filename="package://diablo_bot/meshes/l_wrist_Link.STL" />
-      </geometry>
-      <material
-        name="">
-        <color
-          rgba="0.752941176470588 0.752941176470588 0.752941176470588 1" />
-      </material>
-    </visual>
-    <collision>
-      <origin
-        xyz="0 0 0"
-        rpy="0 0 0" />
-      <geometry>
-        <mesh
-          filename="package://diablo_bot/meshes/l_wrist_Link.STL" />
+          filename="$(find diablo_bot)/description/meshes/l_wrist_Link.STL" />
+      </geometry>
+      <material
+        name="">
+        <color
+          rgba="0.752941176470588 0.752941176470588 0.752941176470588 1" />
+      </material>
+    </visual>
+    <collision>
+      <origin
+        xyz="0 0 0"
+        rpy="0 0 0" />
+      <geometry>
+        <mesh
+          filename="$(find diablo_bot)/description/meshes/l_wrist_Link.STL" />
       </geometry>
     </collision>
@@ -304,19 +304,19 @@
       <geometry>
         <mesh
-          filename="package://diablo_bot/meshes/l_mid_base_Link.STL" />
-      </geometry>
-      <material
-        name="">
-        <color
-          rgba="0.752941176470588 0.752941176470588 0.752941176470588 1" />
-      </material>
-    </visual>
-    <collision>
-      <origin
-        xyz="0 0 0"
-        rpy="0 0 0" />
-      <geometry>
-        <mesh
-          filename="package://diablo_bot/meshes/l_mid_base_Link.STL" />
+          filename="$(find diablo_bot)/description/meshes/l_mid_base_Link.STL" />
+      </geometry>
+      <material
+        name="">
+        <color
+          rgba="0.752941176470588 0.752941176470588 0.752941176470588 1" />
+      </material>
+    </visual>
+    <collision>
+      <origin
+        xyz="0 0 0"
+        rpy="0 0 0" />
+      <geometry>
+        <mesh
+          filename="$(find diablo_bot)/description/meshes/l_mid_base_Link.STL" />
       </geometry>
     </collision>
@@ -362,19 +362,19 @@
       <geometry>
         <mesh
-          filename="package://diablo_bot/meshes/l_mid_middle_Link.STL" />
-      </geometry>
-      <material
-        name="">
-        <color
-          rgba="0.752941176470588 0.752941176470588 0.752941176470588 1" />
-      </material>
-    </visual>
-    <collision>
-      <origin
-        xyz="0 0 0"
-        rpy="0 0 0" />
-      <geometry>
-        <mesh
-          filename="package://diablo_bot/meshes/l_mid_middle_Link.STL" />
+          filename="$(find diablo_bot)/description/meshes/l_mid_middle_Link.STL" />
+      </geometry>
+      <material
+        name="">
+        <color
+          rgba="0.752941176470588 0.752941176470588 0.752941176470588 1" />
+      </material>
+    </visual>
+    <collision>
+      <origin
+        xyz="0 0 0"
+        rpy="0 0 0" />
+      <geometry>
+        <mesh
+          filename="$(find diablo_bot)/description/meshes/l_mid_middle_Link.STL" />
       </geometry>
     </collision>
@@ -420,19 +420,19 @@
       <geometry>
         <mesh
-          filename="package://diablo_bot/meshes/l_mid_tip_Link.STL" />
-      </geometry>
-      <material
-        name="">
-        <color
-          rgba="0.752941176470588 0.752941176470588 0.752941176470588 1" />
-      </material>
-    </visual>
-    <collision>
-      <origin
-        xyz="0 0 0"
-        rpy="0 0 0" />
-      <geometry>
-        <mesh
-          filename="package://diablo_bot/meshes/l_mid_tip_Link.STL" />
+          filename="$(find diablo_bot)/description/meshes/l_mid_tip_Link.STL" />
+      </geometry>
+      <material
+        name="">
+        <color
+          rgba="0.752941176470588 0.752941176470588 0.752941176470588 1" />
+      </material>
+    </visual>
+    <collision>
+      <origin
+        xyz="0 0 0"
+        rpy="0 0 0" />
+      <geometry>
+        <mesh
+          filename="$(find diablo_bot)/description/meshes/l_mid_tip_Link.STL" />
       </geometry>
     </collision>
@@ -478,19 +478,19 @@
       <geometry>
         <mesh
-          filename="package://diablo_bot/meshes/l_thumb_base_Link.STL" />
-      </geometry>
-      <material
-        name="">
-        <color
-          rgba="0.752941176470588 0.752941176470588 0.752941176470588 1" />
-      </material>
-    </visual>
-    <collision>
-      <origin
-        xyz="0 0 0"
-        rpy="0 0 0" />
-      <geometry>
-        <mesh
-          filename="package://diablo_bot/meshes/l_thumb_base_Link.STL" />
+          filename="$(find diablo_bot)/description/meshes/l_thumb_base_Link.STL" />
+      </geometry>
+      <material
+        name="">
+        <color
+          rgba="0.752941176470588 0.752941176470588 0.752941176470588 1" />
+      </material>
+    </visual>
+    <collision>
+      <origin
+        xyz="0 0 0"
+        rpy="0 0 0" />
+      <geometry>
+        <mesh
+          filename="$(find diablo_bot)/description/meshes/l_thumb_base_Link.STL" />
       </geometry>
     </collision>
@@ -536,19 +536,19 @@
       <geometry>
         <mesh
-          filename="package://diablo_bot/meshes/l_thumb_middle_Link.STL" />
-      </geometry>
-      <material
-        name="">
-        <color
-          rgba="0.752941176470588 0.752941176470588 0.752941176470588 1" />
-      </material>
-    </visual>
-    <collision>
-      <origin
-        xyz="0 0 0"
-        rpy="0 0 0" />
-      <geometry>
-        <mesh
-          filename="package://diablo_bot/meshes/l_thumb_middle_Link.STL" />
+          filename="$(find diablo_bot)/description/meshes/l_thumb_middle_Link.STL" />
+      </geometry>
+      <material
+        name="">
+        <color
+          rgba="0.752941176470588 0.752941176470588 0.752941176470588 1" />
+      </material>
+    </visual>
+    <collision>
+      <origin
+        xyz="0 0 0"
+        rpy="0 0 0" />
+      <geometry>
+        <mesh
+          filename="$(find diablo_bot)/description/meshes/l_thumb_middle_Link.STL" />
       </geometry>
     </collision>
@@ -594,19 +594,19 @@
       <geometry>
         <mesh
-          filename="package://diablo_bot/meshes/l_thumb_tip_Link.STL" />
-      </geometry>
-      <material
-        name="">
-        <color
-          rgba="0.752941176470588 0.752941176470588 0.752941176470588 1" />
-      </material>
-    </visual>
-    <collision>
-      <origin
-        xyz="0 0 0"
-        rpy="0 0 0" />
-      <geometry>
-        <mesh
-          filename="package://diablo_bot/meshes/l_thumb_tip_Link.STL" />
+          filename="$(find diablo_bot)/description/meshes/l_thumb_tip_Link.STL" />
+      </geometry>
+      <material
+        name="">
+        <color
+          rgba="0.752941176470588 0.752941176470588 0.752941176470588 1" />
+      </material>
+    </visual>
+    <collision>
+      <origin
+        xyz="0 0 0"
+        rpy="0 0 0" />
+      <geometry>
+        <mesh
+          filename="$(find diablo_bot)/description/meshes/l_thumb_tip_Link.STL" />
       </geometry>
     </collision>
@@ -652,19 +652,19 @@
       <geometry>
         <mesh
-          filename="package://diablo_bot/meshes/l_index_base_Link.STL" />
-      </geometry>
-      <material
-        name="">
-        <color
-          rgba="0.752941176470588 0.752941176470588 0.752941176470588 1" />
-      </material>
-    </visual>
-    <collision>
-      <origin
-        xyz="0 0 0"
-        rpy="0 0 0" />
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
File: description/gazebo_control.xacro (robot description, xacro)
@@ -5,5 +5,5 @@
             <left_joint>l4</left_joint>
             <right_joint>r4</right_joint>
-            <wheel_seperation>0.35</wheel_seperation>
+            <wheel_separation>0.5</wheel_separation>
             <wheel_diameter>0.1</wheel_diameter>
             <max_wheel_torque>200</max_wheel_torque>

File: description/robot.urdf.xacro (robot description, xacro)
@@ -1,12 +1,5 @@
 <?xml version="1.0"?>
 <robot xmlns:xacro="http://www.ros.org/wiki/xacro"  name="diablo_robot">
-    <xacro:arg name="use_ros2_control" default="true"/>
-    <xacro:arg name="sim_mode" default="false"/>
     <xacro:include filename="diablo_core.xacro" />
-    <xacro:if value="$(arg use_ros2_control)">
-        <xacro:include filename="ros2_control.xacro" />
-    </xacro:if>
-    <xacro:unless value="$(arg use_ros2_control)">
-        <xacro:include filename="gazebo_control.xacro" />
-    </xacro:unless>
+    <xacro:include filename="ros2_control.xacro" />
 </robot>

Commit message: diablo_core.xacro

File: description/diablo_core.xacro (robot description, xacro)
@@ -1150,17 +1150,4 @@
       velocity="4.71" />
   </joint>
-  <!-- <joint name="panda_grip_vis_joint" type="fixed">
-    <parent link="r_wrist_Link"/>
-    <child link="panda_grip_site"/>
-    <origin rpy="0 0 0" xyz="0.02 0 0.1125"/>
-  </joint>
-  <link name="panda_grip_site">
-    <visual>
-      <geometry>
-        <sphere radius="0.005"/>
-      </geometry>
-      <material name="Vis"/>
-    </visual>
-  </link> -->
   <link
     name="r_index_base_Link">

Commit message: Added Controller file

File: description/diablo_core.xacro (robot description, xacro)
@@ -1716,5 +1716,5 @@
     <axis xyz="0.0 -1.0 0.0"/>
     <limit  effort="9.6" velocity="12.05"/>
-    <dynamics damping="0" friction="0.1"/>   <!--changed [friction:0]-->
+    <dynamics damping="0" friction="0"/>   <!--changed [friction:0]-->
   </joint>
   <link name="motor_right_link_1">
@@ -1939,5 +1939,5 @@
     <parent link="leg2_right_link_1"/>
     <child link="wheel_right_link_1"/>
-    <axis xyz="0.0 -1.0 -0.0"/>
+    <axis xyz="0.0 -1.0 0.0"/>
     <limit  effort="9.6" velocity="12.05"/>
     <dynamics damping="0" friction="0"/>

File: description/ros2_control.xacro (robot description, xacro)
@@ -1,5 +1,5 @@
 <?xml version="1.0"?>
 <robot xmlns:xacro="http://www.ros.org/wiki/xacro">
-    <transmission name= "l4_trans">
+    <!--<transmission name= "l4_trans">
         <type>transmission_interface/SimpleTransmission</type>
         <joint name='l4'>
@@ -12,29 +12,123 @@
             <hardwareInterface>hardware_interface/VelocityJointInterface</hardwareInterface>
         </joint>
-    </transmission>
-    <ros2_control name="GazeboSystem" type="System">
+    </transmission> -->
+    <ros2_control name="GazeboSystem" type="system">
         <hardware>
-            <plugin> gazebo_ros2_control/GazeboSystem</plugin>
+            <plugin>gazebo_ros2_control/GazeboSystem</plugin>
         </hardware>
+        <!--lower body joints-->
+        <joint name="l_sho_pitch">
+            <command_interface name="position" />
+            <state_interface name='position'>
+                <param name="initial_value">0.0</param>
+            </state_interface>
+            <state_interface name='velocity' />
+        </joint>
+        <joint name="l_sho_roll">
+            <command_interface name="position" />
+            <state_interface name='position'>
+                <param name="initial_value">0.0</param>
+            </state_interface>
+            <state_interface name='velocity' />
+        </joint>
+        <joint name="l_el">
+            <command_interface name="position" />
+            <state_interface name='position'>
+                <param name="initial_value">0.0</param>
+            </state_interface>
+            <state_interface name='velocity' />
+        </joint>
+        <joint name="r_sho_pitch">
+            <command_interface name="position" />
+            <state_interface name='position'>
+                <param name="initial_value">0.0</param>
+            </state_interface>
+            <state_interface name='velocity' />
+        </joint>
+        <joint name="r_sho_roll">
+            <command_interface name="position" />
+            <state_interface name='position'>
+                <param name="initial_value">0.0</param>
+            </state_interface>
+            <state_interface name='velocity' />
+        </joint>
+        <joint name="r_el">
+            <command_interface name="position" />
+            <state_interface name='position'>
+                <param name="initial_value">0.0</param>
+            </state_interface>
+            <state_interface name='velocity' />
+        </joint>
+        <joint name="lower_base_joint">
+            <command_interface name="position" />
+            <state_interface name='position'>
+                <param name="initial_value">0.0</param>
+            </state_interface>
+        </joint>
+        <!--Upper body joints-->
+        <joint name="l1">
+            <command_interface name="position" />
+            <state_interface name='position'>
+                <param name="initial_value">0.0</param>
+            </state_interface>
+            <state_interface name='velocity' />
+        </joint>
+        <joint name="l2">
+            <command_interface name="position" />
+            <state_interface name='position'>
+                <param name="initial_value">0.0</param>
+            </state_interface>
+        </joint>
+        <joint name="l3">
+            <command_interface name="position" />
+            <state_interface name='position'>
+                <param name="initial_value">0.0</param>
+            </state_interface>
+            <state_interface name='velocity' />
+        </joint>
         <joint name="l4">
-            <command_interface name="velocity">
-                <param name="min">-1</param>
-                <param name="max">1</param>
-            </command_interface>
+            <command_interface name="position" />
+            <command_interface name="velocity" />
+            <state_interface name='position'>
+                <param name="initial_value">0.0</param>
+            </state_interface>
+            <state_interface name='velocity'>
+                <param name="initial_value">0.0</param>
+            </state_interface>
+        </joint>
+        <joint name="r1">
+            <command_interface name="position" />
+            <state_interface name='position'>
+                <param name="initial_value">0.0</param>
+            </state_interface>
             <state_interface name='velocity' />
-            <state_interface name='position' />
+        </joint>
+        <joint name="r2">
+            <command_interface name="position" />
+            <state_interface name='position'>
+                <param name="initial_value">0.0</param>
+            </state_interface>
+        </joint>
+        <joint name="r3">
+            <command_interface name="position" />
+            <state_interface name='position'>
+                <param name="initial_value">0.0</param>
+            </state_interface>
+            <state_interface name='velocity' />
         </joint>
         <joint name="r4">
-            <command_interface name="velocity">
-                <param name="min">-1</param>
-                <param name="max">1</param>
-            </command_interface>
-            <state_interface name='velocity' />
-            <state_interface name='position' />
+            <command_interface name="position" />
+            <command_interface name="velocity" />
+            <state_interface name='position'>
+                <param name="initial_value">0.0</param>
+            </state_interface>
+            <state_interface name='velocity'>
+                <param name="initial_value">0.0</param>
+            </state_interface>
         </joint>
     </ros2_control>
     <gazebo>
         <plugin name="gazebo_ros2_control" filename="libgazebo_ros2_control.so">
-            <parameters>$(find diablo_bot)/config/diff_drive_controller.yaml</parameters>
+            <parameters>$(find diablo_bot)/config/my_controllers.yaml</parameters>
         </plugin>
     </gazebo>
