Commit message: Updated config file

File: description/diablo_core.xacro (robot description, xacro)
@@ -14,5 +14,5 @@
         rpy="0 0 0" />
       <mass
-        value="0.459362407581758" />
+        value="0.459362407581758"/>
       <inertia
         ixx="0.00098999304970947"
@@ -21,10 +21,10 @@
         iyy="0.000787503978866051"
         iyz="1.94259853491067E-13"
-        izz="0.000705078033251521" />
-    </inertial>
-    <visual>
-      <origin
-        xyz="0 0 0"
-        rpy="0 0 0" />
+        izz="0.000705078033251521"/>
+    </inertial>
+    <visual>
+      <origin
+        xyz="0 0 0"
+        rpy="0 0 0"/>
       <geometry>
         <mesh
@@ -1716,5 +1716,5 @@
     <axis xyz="0.0 -1.0 0.0"/>
     <limit  effort="9.6" velocity="12.05"/>
-    <dynamics damping="0" friction="0"/>   <!--changed [friction:0]-->
+    <dynamics damping="0" friction="0"/>
   </joint>
   <link name="motor_right_link_1">
@@ -1741,5 +1741,5 @@
     <inertial>
       <origin rpy="0 0 0" xyz="4.148993296440801e-07 0.06735128629132996 -0.0012035359325800465"/>
-      <mass value="4.6"/>
+      <mass value="2.6"/>
       <inertia ixx="0.027399" ixy="0.0" ixz="0.0" iyy="0.027359" iyz="0.000518" izz="0.026313"/>
     </inertial>
@@ -1879,4 +1879,36 @@
   </link>
     <!-- ==================================== Lower Body Joints ============================= -->
+  <joint name="l1" type="continuous">
+    <origin rpy="0 0 0" xyz="0.00036 0.053553 0.379"/>
+    <parent link="lower_base_link"/>
+    <child link="motor_left_link_1"/>
+    <axis xyz="0.0 1.0 0.0"/>
+    <limit  effort="9.6" velocity="12.05"/>
+    <dynamics damping="0" friction="0"/>
+  </joint>
+  <joint name="l2" type="fixed">
+    <origin rpy="0 0 0" xyz="0.0 0.1181 0.0"/>
+    <parent link="motor_left_link_1"/>
+    <child link="leg_left_link_1"/>
+    <axis xyz="0.0 1.0 0.0"/>
+    <limit  effort="9.6" velocity="12.05"/>
+    <dynamics damping="0" friction="0"/>
+  </joint>
+  <joint name="l3" type="continuous">
+    <origin rpy="0 0 0" xyz="0.0 0.016 -0.14"/>
+    <parent link="leg_left_link_1"/>
+    <child link="leg2_left_link_1"/>
+    <axis xyz="0.0 1.0 -0.0"/>
+    <limit  effort="9.6" velocity="12.05"/>
+    <dynamics damping="0" friction="0"/>
+  </joint>
+  <joint name="l4" type="continuous">
+    <origin rpy="0 0 0" xyz="0.0 0.0277 -0.14"/>
+    <parent link="leg2_left_link_1"/>
+    <child link="wheel_left_link_1"/>
+    <axis xyz="0.0 1.0 0.0"/>
+    <limit  effort="9.6" velocity="12.05"/>
+    <dynamics damping="0" friction="0"/>
+  </joint>
   <joint name="r1" type="continuous">
     <origin rpy="0 0 0" xyz="0.00036 -0.053347 0.379"/>
@@ -1887,36 +1919,4 @@
     <dynamics damping="0" friction="0"/>
   </joint>
-  <joint name="l1" type="continuous">
-    <origin rpy="0 0 0" xyz="0.00036 0.053553 0.379"/>
-    <parent link="lower_base_link"/>
-    <child link="motor_left_link_1"/>
-    <axis xyz="0.0 1.0 0.0"/>
-    <limit  effort="9.6" velocity="12.05"/>
-    <dynamics damping="0" friction="0"/>
-  </joint>
-  <joint name="l2" type="fixed">
-    <origin rpy="0 0 0" xyz="0.0 0.1181 0.0"/>
-    <parent link="motor_left_link_1"/>
-    <child link="leg_left_link_1"/>
-    <axis xyz="0.0 1.0 0.0"/>
-    <limit  effort="9.6" velocity="12.05"/>
-    <dynamics damping="0" friction="0"/>
-  </joint>
-  <joint name="l3" type="continuous">
-    <origin rpy="0 0 0" xyz="0.0 0.016 -0.14"/>
-    <parent link="leg_left_link_1"/>
-    <child link="leg2_left_link_1"/>
-    <axis xyz="0.0 1.0 -0.0"/>
-    <limit  effort="9.6" velocity="12.05"/>
-    <dynamics damping="0" friction="0"/>
-  </joint>
-  <joint name="l4" type="continuous">
-    <origin rpy="0 0 0" xyz="0.0 0.0277 -0.14"/>
-    <parent link="leg2_left_link_1"/>
-    <child link="wheel_left_link_1"/>
-    <axis xyz="0.0 1.0 0.0"/>
-    <limit  effort="9.6" velocity="12.05"/>
-    <dynamics damping="0" friction="0"/>
-  </joint>
   <joint name="r2" type="fixed">
     <origin rpy="0 0 0" xyz="0.0 -0.1181 0.0"/>

File: description/ros2_control.xacro (robot description, xacro)
@@ -1,21 +1,9 @@
 <?xml version="1.0"?>
 <robot xmlns:xacro="http://www.ros.org/wiki/xacro">
-    <!--<transmission name= "l4_trans">
-        <type>transmission_interface/SimpleTransmission</type>
-        <joint name='l4'>
-            <hardwareInterface>hardware_interface/VelocityJointInterface</hardwareInterface>
-        </joint>
-    </transmission>
-    <transmission name= "r4_trans">
-        <type>transmission_interface/SimpleTransmission</type>
-        <joint name='r4'>
-            <hardwareInterface>hardware_interface/VelocityJointInterface</hardwareInterface>
-        </joint>
-    </transmission> -->
     <ros2_control name="GazeboSystem" type="system">
         <hardware>
             <plugin>gazebo_ros2_control/GazeboSystem</plugin>
         </hardware>
-        <!--lower body joints-->
+        <!--Upper body joints-->
         <joint name="l_sho_pitch">
             <command_interface name="position" />
@@ -66,11 +54,13 @@
             </state_interface>
         </joint>
-        <!--Upper body joints-->
+        <!--lower body joints-->
         <joint name="l1">
-            <command_interface name="position" />
-            <state_interface name='position'>
-                <param name="initial_value">0.0</param>
-            </state_interface>
-            <state_interface name='velocity' />
+            <command_interface name="position">
+                <param name="min">-3.14</param>
+                <param name="max">3.14</param>
+            </command_interface>
+            <state_interface name="position"/>
+            <state_interface name="velocity"/>
+            <state_interface name="effort"/>
         </joint>
         <joint name="l2">
@@ -81,26 +71,29 @@
         </joint>
         <joint name="l3">
-            <command_interface name="position" />
-            <state_interface name='position'>
-                <param name="initial_value">0.0</param>
-            </state_interface>
-            <state_interface name='velocity' />
+            <command_interface name="position">
+                <param name="min">-3.14</param>
+                <param name="max">3.14</param>
+            </command_interface>
+            <state_interface name="position"/>
+            <state_interface name="velocity"/>
+            <state_interface name="effort"/>
         </joint>
         <joint name="l4">
-            <command_interface name="position" />
-            <command_interface name="velocity" />
-            <state_interface name='position'>
-                <param name="initial_value">0.0</param>
-            </state_interface>
-            <state_interface name='velocity'>
-                <param name="initial_value">0.0</param>
-            </state_interface>
+            <command_interface name="velocity">
+                <param name="min">-1.0</param>
+                <param name="max">1.0</param>
+            </command_interface>
+            <state_interface name='position'/>
+            <state_interface name='velocity'/>
+            <state_interface name='effort'/>
         </joint>
         <joint name="r1">
-            <command_interface name="position" />
-            <state_interface name='position'>
-                <param name="initial_value">0.0</param>
-            </state_interface>
-            <state_interface name='velocity' />
+            <command_interface name="position">
+                <param name="min">-3.14</param>
+                <param name="max">3.14</param>
+            </command_interface>
+            <state_interface name="position"/>
+            <state_interface name="velocity"/>
+            <state_interface name="effort"/>
         </joint>
         <joint name="r2">
@@ -111,19 +104,20 @@
         </joint>
         <joint name="r3">
-            <command_interface name="position" />
-            <state_interface name='position'>
-                <param name="initial_value">0.0</param>
-            </state_interface>
-            <state_interface name='velocity' />
+            <command_interface name="position">
+                <param name="min">-3.14</param>
+                <param name="max">3.14</param>
+            </command_interface>
+            <state_interface name="position"/>
+            <state_interface name="velocity"/>
+            <state_interface name="effort"/>
         </joint>
         <joint name="r4">
-            <command_interface name="position" />
-            <command_interface name="velocity" />
-            <state_interface name='position'>
-                <param name="initial_value">0.0</param>
-            </state_interface>
-            <state_interface name='velocity'>
-                <param name="initial_value">0.0</param>
-            </state_interface>
+            <command_interface name="velocity">
+                <param name="min">-1.0</param>
+                <param name="max">1.0</param>
+            </command_interface>
+            <state_interface name='position'/>
+            <state_interface name='velocity'/>
+            <state_interface name='effort'/>
         </joint>
     </ros2_control>

Commit message: Modified .yaml file

File: description/diablo_core.xacro (robot description, xacro)
@@ -1710,5 +1710,5 @@
     </collision>
   </link>
-  <joint name="lower_base_joint" type="fixed">
+    <joint name="lower_base_joint" type="fixed">
     <origin rpy="0 0 0" xyz="0.0 0.0 -0.5"/>
     <parent link="base_link"/>
@@ -1741,5 +1741,5 @@
     <inertial>
       <origin rpy="0 0 0" xyz="4.148993296440801e-07 0.06735128629132996 -0.0012035359325800465"/>
-      <mass value="2.6"/>
+      <mass value="4.6"/>
       <inertia ixx="0.027399" ixy="0.0" ixz="0.0" iyy="0.027359" iyz="0.000518" izz="0.026313"/>
     </inertial>
@@ -1878,6 +1878,13 @@
     </collision>
   </link>
-    <!-- ==================================== Lower Body Joints ============================= -->
-  <joint name="l1" type="continuous">
+  <joint name="r1" type="continous">
+    <origin rpy="0 0 0" xyz="0.00036 -0.053347 0.379"/>
+    <parent link="lower_base_link"/>
+    <child link="motor_right_link_1"/>
+    <axis xyz="0.0 -1.0 0.0"/>
+    <limit  effort="9.6" velocity="12.05"/>
+    <dynamics damping="0" friction="0"/>
+  </joint>
+  <joint name="l1" type="continous">
     <origin rpy="0 0 0" xyz="0.00036 0.053553 0.379"/>
     <parent link="lower_base_link"/>
@@ -1895,28 +1902,4 @@
     <dynamics damping="0" friction="0"/>
   </joint>
-  <joint name="l3" type="continuous">
-    <origin rpy="0 0 0" xyz="0.0 0.016 -0.14"/>
-    <parent link="leg_left_link_1"/>
-    <child link="leg2_left_link_1"/>
-    <axis xyz="0.0 1.0 -0.0"/>
-    <limit  effort="9.6" velocity="12.05"/>
-    <dynamics damping="0" friction="0"/>
-  </joint>
-  <joint name="l4" type="continuous">
-    <origin rpy="0 0 0" xyz="0.0 0.0277 -0.14"/>
-    <parent link="leg2_left_link_1"/>
-    <child link="wheel_left_link_1"/>
-    <axis xyz="0.0 1.0 0.0"/>
-    <limit  effort="9.6" velocity="12.05"/>
-    <dynamics damping="0" friction="0"/>
-  </joint>
-  <joint name="r1" type="continuous">
-    <origin rpy="0 0 0" xyz="0.00036 -0.053347 0.379"/>
-    <parent link="lower_base_link"/>
-    <child link="motor_right_link_1"/>
-    <axis xyz="0.0 -1.0 0.0"/>
-    <limit  effort="9.6" velocity="12.05"/>
-    <dynamics damping="0" friction="0"/>
-  </joint>
   <joint name="r2" type="fixed">
     <origin rpy="0 0 0" xyz="0.0 -0.1181 0.0"/>
@@ -1927,5 +1910,13 @@
     <dynamics damping="0" friction="0"/>
   </joint>
-  <joint name="r3" type="continuous">
+  <joint name="l3" type="continous">
+    <origin rpy="0 0 0" xyz="0.0 0.016 -0.14"/>
+    <parent link="leg_left_link_1"/>
+    <child link="leg2_left_link_1"/>
+    <axis xyz="0.0 1.0 0.0"/>
+    <limit  effort="9.6" velocity="12.05"/>
+    <dynamics damping="0" friction="0"/>
+  </joint>
+  <joint name="r3" type="continous">
     <origin rpy="0 0 0" xyz="0.0 -0.016 -0.14"/>
     <parent link="leg_right_link_1"/>
@@ -1935,9 +1926,17 @@
     <dynamics damping="0" friction="0"/>
   </joint>
-  <joint name="r4" type="continuous">
+  <joint name="l4" type="continous">
+    <origin rpy="0 0 0" xyz="0.0 0.0277 -0.14"/>
+    <parent link="leg2_left_link_1"/>
+    <child link="wheel_left_link_1"/>
+    <axis xyz="0.0 1.0 0.0"/>
+    <limit  effort="9.6" velocity="12.05"/>
+    <dynamics damping="0" friction="0"/>
+  </joint>
+  <joint name="r4" type="continous">
     <origin rpy="0 0 0" xyz="0.0 -0.0277 -0.14"/>
     <parent link="leg2_right_link_1"/>
     <child link="wheel_right_link_1"/>
-    <axis xyz="0.0 -1.0 0.0"/>
+    <axis xyz="0.0 -1.0 -0.0"/>
     <limit  effort="9.6" velocity="12.05"/>
     <dynamics damping="0" friction="0"/>

File: description/ros2_control.xacro (robot description, xacro)
@@ -6,4 +6,38 @@
         </hardware>
         <!--Upper body joints-->
+        <joint name="head_pan">
+            <command_interface name="position" />
+            <state_interface name='position'>
+                <param name="initial_value">0.0</param>
+            </state_interface>
+            <state_interface name='velocity' />
+        </joint>
+        <joint name="head_tilt">
+            <command_interface name="position" />
+            <state_interface name='position'>
+                <param name="initial_value">0.0</param>
+            </state_interface>
+            <state_interface name='velocity' />
+        </joint>
+        <joint name="l_wrist">
+        </joint>
+        <joint name="r_wrist">
+        </joint>
+        <joint name="l_index_base">
+        </joint>
+        <joint name="r_index_base">
+        </joint>
+        <joint name="l_index_middle">
+        </joint>
+        <joint name="r_index_middle">
+        </joint>
+        <joint name="l_index_tip">
+        </joint>
+        <joint name="r_index_tip">
+        </joint>
+        <joint name="l_mid_base">
+        </joint>
+        <joint name="r_mid_base">
+        </joint>
         <joint name="l_sho_pitch">
             <command_interface name="position" />
@@ -48,36 +82,38 @@
             <state_interface name='velocity' />
         </joint>
-        <joint name="lower_base_joint">
+        <!--lower body joints-->
+        <joint name="l1">
             <command_interface name="position" />
             <state_interface name='position'>
                 <param name="initial_value">0.0</param>
             </state_interface>
+            <state_interface name='velocity'/>
+            <state_interface name='effort'/>
         </joint>
-        <!--lower body joints-->
-        <joint name="l1">
-            <command_interface name="position">
-                <param name="min">-3.14</param>
-                <param name="max">3.14</param>
-            </command_interface>
-            <state_interface name="position"/>
-            <state_interface name="velocity"/>
-            <state_interface name="effort"/>
-        </joint>
-        <joint name="l2">
+        <joint name="r1">
             <command_interface name="position" />
             <state_interface name='position'>
                 <param name="initial_value">0.0</param>
             </state_interface>
+            <state_interface name='velocity'/>
+            <state_interface name='effort'/>
         </joint>
         <joint name="l3">
-            <command_interface name="position">
-                <param name="min">-3.14</param>
-                <param name="max">3.14</param>
-            </command_interface>
-            <state_interface name="position"/>
-            <state_interface name="velocity"/>
-            <state_interface name="effort"/>
+            <command_interface name="position" />
+            <state_interface name='position'>
+                <param name="initial_value">0.0</param>
+            </state_interface>
+            <state_interface name='velocity'/>
+            <state_interface name='effort'/>
         </joint>
-        <joint name="l4">
+        <joint name="r3">
+            <command_interface name='position' />
+            <state_interface name='position'>
+                <param name="initial_value">0.0</param>
+            </state_interface>
+            <state_interface name='velocity'/>
+            <state_interface name='effort'/>
+        </joint>
+        <joint name="r4">
             <command_interface name="velocity">
                 <param name="min">-1.0</param>
@@ -88,29 +124,5 @@
             <state_interface name='effort'/>
         </joint>
-        <joint name="r1">
-            <command_interface name="position">
-                <param name="min">-3.14</param>
-                <param name="max">3.14</param>
-            </command_interface>
-            <state_interface name="position"/>
-            <state_interface name="velocity"/>
-            <state_interface name="effort"/>
-        </joint>
-        <joint name="r2">
-            <command_interface name="position" />
-            <state_interface name='position'>
-                <param name="initial_value">0.0</param>
-            </state_interface>
-        </joint>
-        <joint name="r3">
-            <command_interface name="position">
-                <param name="min">-3.14</param>
-                <param name="max">3.14</param>
-            </command_interface>
-            <state_interface name="position"/>
-            <state_interface name="velocity"/>
-            <state_interface name="effort"/>
-        </joint>
-        <joint name="r4">
+        <joint name="l4">
             <command_interface name="velocity">
                 <param name="min">-1.0</param>

Commit message: modified .yaml file

File: description/diablo_core.xacro (robot description, xacro)
@@ -1878,5 +1878,5 @@
     </collision>
   </link>
-  <joint name="r1" type="continous">
+  <joint name="r1" type="continuous ">
     <origin rpy="0 0 0" xyz="0.00036 -0.053347 0.379"/>
     <parent link="lower_base_link"/>
@@ -1886,5 +1886,5 @@
     <dynamics damping="0" friction="0"/>
   </joint>
-  <joint name="l1" type="continous">
+  <joint name="l1" type="continuous ">
     <origin rpy="0 0 0" xyz="0.00036 0.053553 0.379"/>
     <parent link="lower_base_link"/>
@@ -1910,5 +1910,5 @@
     <dynamics damping="0" friction="0"/>
   </joint>
-  <joint name="l3" type="continous">
+  <joint name="l3" type="continuous">
     <origin rpy="0 0 0" xyz="0.0 0.016 -0.14"/>
     <parent link="leg_left_link_1"/>
@@ -1918,5 +1918,5 @@
     <dynamics damping="0" friction="0"/>
   </joint>
-  <joint name="r3" type="continous">
+  <joint name="r3" type="continuous">
     <origin rpy="0 0 0" xyz="0.0 -0.016 -0.14"/>
     <parent link="leg_right_link_1"/>
@@ -1926,5 +1926,5 @@
     <dynamics damping="0" friction="0"/>
   </joint>
-  <joint name="l4" type="continous">
+  <joint name="l4" type="continuous">
     <origin rpy="0 0 0" xyz="0.0 0.0277 -0.14"/>
     <parent link="leg2_left_link_1"/>
@@ -1934,5 +1934,5 @@
     <dynamics damping="0" friction="0"/>
   </joint>
-  <joint name="r4" type="continous">
+  <joint name="r4" type="continuous">
     <origin rpy="0 0 0" xyz="0.0 -0.0277 -0.14"/>
     <parent link="leg2_right_link_1"/>

Commit message: Update diablo_core.xacro

File: description/diablo_core.xacro (robot description, xacro)
@@ -1878,5 +1878,5 @@
     </collision>
   </link>
-  <joint name="r1" type="continuous ">
+  <joint name="r1" type="continuous">
     <origin rpy="0 0 0" xyz="0.00036 -0.053347 0.379"/>
     <parent link="lower_base_link"/>
@@ -1886,5 +1886,5 @@
     <dynamics damping="0" friction="0"/>
   </joint>
-  <joint name="l1" type="continuous ">
+  <joint name="l1" type="continuous">
     <origin rpy="0 0 0" xyz="0.00036 0.053553 0.379"/>
     <parent link="lower_base_link"/>
