Commit message: Added IMU sensor

File: description/diablo_core.xacro (robot description, xacro)
@@ -7,4 +7,9 @@
 <!-- |                                      UPPER BODY                                 | -->
 <!-- =================================================================================== -->
+  <link name="dummy_root"/>
+  <joint name="dummy_to_base" type="fixed">
+    <parent link="dummy_root"/>
+    <child link="base_link"/>
+  </joint>
   <link
     name="base_link">
@@ -29,19 +34,19 @@
       <geometry>
         <mesh
-          filename="$(find diablo_bot)/description/meshes/base_link.STL" />
-      </geometry>
-      <material
-        name="">
-        <color
-          rgba="0.752941176470588 0.752941176470588 0.752941176470588 1" />
-      </material>
-    </visual>
-    <collision>
-      <origin
-        xyz="0 0 0"
-        rpy="0 0 0" />
-      <geometry>
-        <mesh
-          filename="$(find diablo_bot)/description/meshes/base_link.STL" />
+          filename="package://diablo_bot/description/meshes/base_link.STL" />
+      </geometry>
+      <material
+        name="">
+        <color
+          rgba="0.752941176470588 0.752941176470588 0.752941176470588 1" />
+      </material>
+    </visual>
+    <collision>
+      <origin
+        xyz="0 0 0"
+        rpy="0 0 0" />
+      <geometry>
+        <mesh
+          filename="package://diablo_bot/description/meshes/base_link.STL" />
       </geometry>
     </collision>
@@ -72,19 +77,19 @@
       <geometry>
         <mesh
-          filename="$(find diablo_bot)/description/meshes/l_sho_pitch_Link.STL" />
-      </geometry>
-      <material
-        name="">
-        <color
-          rgba="0.752941176470588 0.752941176470588 0.752941176470588 1" />
-      </material>
-    </visual>
-    <collision>
-      <origin
-        xyz="0 0 0"
-        rpy="0 0 0" />
-      <geometry>
-        <mesh
-          filename="$(find diablo_bot)/description/meshes/l_sho_pitch_Link.STL" />
+          filename="package://diablo_bot/description/meshes/l_sho_pitch_Link.STL" />
+      </geometry>
+      <material
+        name="">
+        <color
+          rgba="0.752941176470588 0.752941176470588 0.752941176470588 1" />
+      </material>
+    </visual>
+    <collision>
+      <origin
+        xyz="0 0 0"
+        rpy="0 0 0" />
+      <geometry>
+        <mesh
+          filename="package://diablo_bot/description/meshes/l_sho_pitch_Link.STL" />
       </geometry>
     </collision>
@@ -130,19 +135,19 @@
       <geometry>
         <mesh
-          filename="$(find diablo_bot)/description/meshes/l_sho_roll_Link.STL" />
-      </geometry>
-      <material
-        name="">
-        <color
-          rgba="0.752941176470588 0.752941176470588 0.752941176470588 1" />
-      </material>
-    </visual>
-    <collision>
-      <origin
-        xyz="0 0 0"
-        rpy="0 0 0" />
-      <geometry>
-        <mesh
-          filename="$(find diablo_bot)/description/meshes/l_sho_roll_Link.STL" />
+          filename="package://diablo_bot/description/meshes/l_sho_roll_Link.STL" />
+      </geometry>
+      <material
+        name="">
+        <color
+          rgba="0.752941176470588 0.752941176470588 0.752941176470588 1" />
+      </material>
+    </visual>
+    <collision>
+      <origin
+        xyz="0 0 0"
+        rpy="0 0 0" />
+      <geometry>
+        <mesh
+          filename="package://diablo_bot/description/meshes/l_sho_roll_Link.STL" />
       </geometry>
     </collision>
@@ -188,19 +193,19 @@
       <geometry>
         <mesh
-          filename="$(find diablo_bot)/description/meshes/l_el_Link.STL" />
-      </geometry>
-      <material
-        name="">
-        <color
-          rgba="0.752941176470588 0.752941176470588 0.752941176470588 1" />
-      </material>
-    </visual>
-    <collision>
-      <origin
-        xyz="0 0 0"
-        rpy="0 0 0" />
-      <geometry>
-        <mesh
-          filename="$(find diablo_bot)/description/meshes/l_el_Link.STL" />
+          filename="package://diablo_bot/description/meshes/l_el_Link.STL" />
+      </geometry>
+      <material
+        name="">
+        <color
+          rgba="0.752941176470588 0.752941176470588 0.752941176470588 1" />
+      </material>
+    </visual>
+    <collision>
+      <origin
+        xyz="0 0 0"
+        rpy="0 0 0" />
+      <geometry>
+        <mesh
+          filename="package://diablo_bot/description/meshes/l_el_Link.STL" />
       </geometry>
     </collision>
@@ -246,19 +251,19 @@
       <geometry>
         <mesh
-          filename="$(find diablo_bot)/description/meshes/l_wrist_Link.STL" />
-      </geometry>
-      <material
-        name="">
-        <color
-          rgba="0.752941176470588 0.752941176470588 0.752941176470588 1" />
-      </material>
-    </visual>
-    <collision>
-      <origin
-        xyz="0 0 0"
-        rpy="0 0 0" />
-      <geometry>
-        <mesh
-          filename="$(find diablo_bot)/description/meshes/l_wrist_Link.STL" />
+          filename="package://diablo_bot/description/meshes/l_wrist_Link.STL" />
+      </geometry>
+      <material
+        name="">
+        <color
+          rgba="0.752941176470588 0.752941176470588 0.752941176470588 1" />
+      </material>
+    </visual>
+    <collision>
+      <origin
+        xyz="0 0 0"
+        rpy="0 0 0" />
+      <geometry>
+        <mesh
+          filename="package://diablo_bot/description/meshes/l_wrist_Link.STL" />
       </geometry>
     </collision>
@@ -304,19 +309,19 @@
       <geometry>
         <mesh
-          filename="$(find diablo_bot)/description/meshes/l_mid_base_Link.STL" />
-      </geometry>
-      <material
-        name="">
-        <color
-          rgba="0.752941176470588 0.752941176470588 0.752941176470588 1" />
-      </material>
-    </visual>
-    <collision>
-      <origin
-        xyz="0 0 0"
-        rpy="0 0 0" />
-      <geometry>
-        <mesh
-          filename="$(find diablo_bot)/description/meshes/l_mid_base_Link.STL" />
+          filename="package://diablo_bot/description/meshes/l_mid_base_Link.STL" />
+      </geometry>
+      <material
+        name="">
+        <color
+          rgba="0.752941176470588 0.752941176470588 0.752941176470588 1" />
+      </material>
+    </visual>
+    <collision>
+      <origin
+        xyz="0 0 0"
+        rpy="0 0 0" />
+      <geometry>
+        <mesh
+          filename="package://diablo_bot/description/meshes/l_mid_base_Link.STL" />
       </geometry>
     </collision>
@@ -362,19 +367,19 @@
       <geometry>
         <mesh
-          filename="$(find diablo_bot)/description/meshes/l_mid_middle_Link.STL" />
-      </geometry>
-      <material
-        name="">
-        <color
-          rgba="0.752941176470588 0.752941176470588 0.752941176470588 1" />
-      </material>
-    </visual>
-    <collision>
-      <origin
-        xyz="0 0 0"
-        rpy="0 0 0" />
-      <geometry>
-        <mesh
-          filename="$(find diablo_bot)/description/meshes/l_mid_middle_Link.STL" />
+          filename="package://diablo_bot/description/meshes/l_mid_middle_Link.STL" />
+      </geometry>
+      <material
+        name="">
+        <color
+          rgba="0.752941176470588 0.752941176470588 0.752941176470588 1" />
+      </material>
+    </visual>
+    <collision>
+      <origin
+        xyz="0 0 0"
+        rpy="0 0 0" />
+      <geometry>
+        <mesh
+          filename="package://diablo_bot/description/meshes/l_mid_middle_Link.STL" />
       </geometry>
     </collision>
@@ -420,19 +425,19 @@
       <geometry>
         <mesh
-          filename="$(find diablo_bot)/description/meshes/l_mid_tip_Link.STL" />
-      </geometry>
-      <material
-        name="">
-        <color
-          rgba="0.752941176470588 0.752941176470588 0.752941176470588 1" />
-      </material>
-    </visual>
-    <collision>
-      <origin
-        xyz="0 0 0"
-        rpy="0 0 0" />
-      <geometry>
-        <mesh
-          filename="$(find diablo_bot)/description/meshes/l_mid_tip_Link.STL" />
+          filename="package://diablo_bot/description/meshes/l_mid_tip_Link.STL" />
+      </geometry>
+      <material
+        name="">
+        <color
+          rgba="0.752941176470588 0.752941176470588 0.752941176470588 1" />
+      </material>
+    </visual>
+    <collision>
+      <origin
+        xyz="0 0 0"
+        rpy="0 0 0" />
+      <geometry>
+        <mesh
+          filename="package://diablo_bot/description/meshes/l_mid_tip_Link.STL" />
       </geometry>
     </collision>
@@ -478,19 +483,19 @@
       <geometry>
         <mesh
-          filename="$(find diablo_bot)/description/meshes/l_thumb_base_Link.STL" />
-      </geometry>
-      <material
-        name="">
-        <color
-          rgba="0.752941176470588 0.752941176470588 0.752941176470588 1" />
-      </material>
-    </visual>
-    <collision>
-      <origin
-        xyz="0 0 0"
-        rpy="0 0 0" />
-      <geometry>
-        <mesh
-          filename="$(find diablo_bot)/description/meshes/l_thumb_base_Link.STL" />
+          filename="package://diablo_bot/description/meshes/l_thumb_base_Link.STL" />
+      </geometry>
+      <material
+        name="">
+        <color
+          rgba="0.752941176470588 0.752941176470588 0.752941176470588 1" />
+      </material>
+    </visual>
+    <collision>
+      <origin
+        xyz="0 0 0"
+        rpy="0 0 0" />
+      <geometry>
+        <mesh
+          filename="package://diablo_bot/description/meshes/l_thumb_base_Link.STL" />
       </geometry>
     </collision>
@@ -536,19 +541,19 @@
       <geometry>
         <mesh
-          filename="$(find diablo_bot)/description/meshes/l_thumb_middle_Link.STL" />
-      </geometry>
-      <material
-        name="">
-        <color
-          rgba="0.752941176470588 0.752941176470588 0.752941176470588 1" />
-      </material>
-    </visual>
-    <collision>
-      <origin
-        xyz="0 0 0"
-        rpy="0 0 0" />
-      <geometry>
-        <mesh
-          filename="$(find diablo_bot)/description/meshes/l_thumb_middle_Link.STL" />
+          filename="package://diablo_bot/description/meshes/l_thumb_middle_Link.STL" />
+      </geometry>
+      <material
+        name="">
+        <color
+          rgba="0.752941176470588 0.752941176470588 0.752941176470588 1" />
+      </material>
+    </visual>
+    <collision>
+      <origin
+        xyz="0 0 0"
+        rpy="0 0 0" />
+      <geometry>
+        <mesh
+          filename="package://diablo_bot/description/meshes/l_thumb_middle_Link.STL" />
       </geometry>
     </collision>
@@ -594,19 +599,19 @@
       <geometry>
         <mesh
-          filename="$(find diablo_bot)/description/meshes/l_thumb_tip_Link.STL" />
-      </geometry>
-      <material
-        name="">
-        <color
-          rgba="0.752941176470588 0.752941176470588 0.752941176470588 1" />
-      </material>
-    </visual>
-    <collision>
-      <origin
-        xyz="0 0 0"
-        rpy="0 0 0" />
-      <geometry>
-        <mesh
-          filename="$(find diablo_bot)/description/meshes/l_thumb_tip_Link.STL" />
+          filename="package://diablo_bot/description/meshes/l_thumb_tip_Link.STL" />
+      </geometry>
+      <material
+        name="">
+        <color
+          rgba="0.752941176470588 0.752941176470588 0.752941176470588 1" />
+      </material>
+    </visual>
+    <collision>
+      <origin
+        xyz="0 0 0"
+        rpy="0 0 0" />
+      <geometry>
+        <mesh
+          filename="package://diablo_bot/description/meshes/l_thumb_tip_Link.STL" />
       </geometry>
     </collision>
@@ -652,19 +657,19 @@
       <geometry>
         <mesh
-          filename="$(find diablo_bot)/description/meshes/l_index_base_Link.STL" />
-      </geometry>
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
File: description/robot.urdf.xacro (robot description, xacro)
@@ -2,4 +2,5 @@
 <robot xmlns:xacro="http://www.ros.org/wiki/xacro"  name="diablo_robot">
     <xacro:include filename="diablo_core.xacro" />
-    <xacro:include filename="ros2_control.xacro" />
+    <!--<xacro:include filename="ros2_control.xacro" />
+    <xacro:include filename="gazebo_plugin.xacro" />-->
 </robot>

File: description/ros2_control.xacro (robot description, xacro)
@@ -6,38 +6,4 @@
         </hardware>
         <!--Upper body joints-->
-        <joint name="head_pan">
-            <command_interface name="position" />
-            <state_interface name='position'>
-                <param name="initial_value">0.0</param>
-            </state_interface>
-            <state_interface name='velocity' />
-        </joint>
-        <joint name="head_tilt">
-            <command_interface name="position" />
-            <state_interface name='position'>
-                <param name="initial_value">0.0</param>
-            </state_interface>
-            <state_interface name='velocity' />
-        </joint>
-        <joint name="l_wrist">
-        </joint>
-        <joint name="r_wrist">
-        </joint>
-        <joint name="l_index_base">
-        </joint>
-        <joint name="r_index_base">
-        </joint>
-        <joint name="l_index_middle">
-        </joint>
-        <joint name="r_index_middle">
-        </joint>
-        <joint name="l_index_tip">
-        </joint>
-        <joint name="r_index_tip">
-        </joint>
-        <joint name="l_mid_base">
-        </joint>
-        <joint name="r_mid_base">
-        </joint>
         <joint name="l_sho_pitch">
             <command_interface name="position" />
@@ -134,8 +100,3 @@
         </joint>
     </ros2_control>
-    <gazebo>
-        <plugin name="gazebo_ros2_control" filename="libgazebo_ros2_control.so">
-            <parameters>$(find diablo_bot)/config/my_controllers.yaml</parameters>
-        </plugin>
-    </gazebo>
 </robot>
