Commit message: Added IMU sensor

File: description/diablo_core.xacro (robot description, xacro)
@@ -7,9 +7,4 @@
 <!-- |                                      UPPER BODY                                 | -->
 <!-- =================================================================================== -->
-  <link name="dummy_root"/>
-  <joint name="dummy_to_base" type="fixed">
-    <parent link="dummy_root"/>
-    <child link="base_link"/>
-  </joint>
   <link
     name="base_link">
@@ -34,19 +29,19 @@
       <geometry>
         <mesh
-          filename="package://diablo_bot/description/meshes/base_link.STL" />
-      </geometry>
-      <material
-        name="">
-        <color
-          rgba="0.752941176470588 0.752941176470588 0.752941176470588 1" />
-      </material>
-    </visual>
-    <collision>
-      <origin
-        xyz="0 0 0"
-        rpy="0 0 0" />
-      <geometry>
-        <mesh
-          filename="package://diablo_bot/description/meshes/base_link.STL" />
+          filename="package://diablo_bot/meshes/base_link.STL" />
+      </geometry>
+      <material
+        name="">
+        <color
+          rgba="0.752941176470588 0.752941176470588 0.752941176470588 1" />
+      </material>
+    </visual>
+    <collision>
+      <origin
+        xyz="0 0 0"
+        rpy="0 0 0" />
+      <geometry>
+        <mesh
+          filename="package://diablo_bot/meshes/base_link.STL" />
       </geometry>
     </collision>
@@ -77,19 +72,19 @@
       <geometry>
         <mesh
-          filename="package://diablo_bot/description/meshes/l_sho_pitch_Link.STL" />
-      </geometry>
-      <material
-        name="">
-        <color
-          rgba="0.752941176470588 0.752941176470588 0.752941176470588 1" />
-      </material>
-    </visual>
-    <collision>
-      <origin
-        xyz="0 0 0"
-        rpy="0 0 0" />
-      <geometry>
-        <mesh
-          filename="package://diablo_bot/description/meshes/l_sho_pitch_Link.STL" />
+          filename="package://diablo_bot/meshes/l_sho_pitch_Link.STL" />
+      </geometry>
+      <material
+        name="">
+        <color
+          rgba="0.752941176470588 0.752941176470588 0.752941176470588 1" />
+      </material>
+    </visual>
+    <collision>
+      <origin
+        xyz="0 0 0"
+        rpy="0 0 0" />
+      <geometry>
+        <mesh
+          filename="package://diablo_bot/meshes/l_sho_pitch_Link.STL" />
       </geometry>
     </collision>
@@ -135,19 +130,19 @@
       <geometry>
         <mesh
-          filename="package://diablo_bot/description/meshes/l_sho_roll_Link.STL" />
-      </geometry>
-      <material
-        name="">
-        <color
-          rgba="0.752941176470588 0.752941176470588 0.752941176470588 1" />
-      </material>
-    </visual>
-    <collision>
-      <origin
-        xyz="0 0 0"
-        rpy="0 0 0" />
-      <geometry>
-        <mesh
-          filename="package://diablo_bot/description/meshes/l_sho_roll_Link.STL" />
+          filename="package://diablo_bot/meshes/l_sho_roll_Link.STL" />
+      </geometry>
+      <material
+        name="">
+        <color
+          rgba="0.752941176470588 0.752941176470588 0.752941176470588 1" />
+      </material>
+    </visual>
+    <collision>
+      <origin
+        xyz="0 0 0"
+        rpy="0 0 0" />
+      <geometry>
+        <mesh
+          filename="package://diablo_bot/meshes/l_sho_roll_Link.STL" />
       </geometry>
     </collision>
@@ -193,19 +188,19 @@
       <geometry>
         <mesh
-          filename="package://diablo_bot/description/meshes/l_el_Link.STL" />
-      </geometry>
-      <material
-        name="">
-        <color
-          rgba="0.752941176470588 0.752941176470588 0.752941176470588 1" />
-      </material>
-    </visual>
-    <collision>
-      <origin
-        xyz="0 0 0"
-        rpy="0 0 0" />
-      <geometry>
-        <mesh
-          filename="package://diablo_bot/description/meshes/l_el_Link.STL" />
+          filename="package://diablo_bot/meshes/l_el_Link.STL" />
+      </geometry>
+      <material
+        name="">
+        <color
+          rgba="0.752941176470588 0.752941176470588 0.752941176470588 1" />
+      </material>
+    </visual>
+    <collision>
+      <origin
+        xyz="0 0 0"
+        rpy="0 0 0" />
+      <geometry>
+        <mesh
+          filename="package://diablo_bot/meshes/l_el_Link.STL" />
       </geometry>
     </collision>
@@ -251,19 +246,19 @@
       <geometry>
         <mesh
-          filename="package://diablo_bot/description/meshes/l_wrist_Link.STL" />
-      </geometry>
-      <material
-        name="">
-        <color
-          rgba="0.752941176470588 0.752941176470588 0.752941176470588 1" />
-      </material>
-    </visual>
-    <collision>
-      <origin
-        xyz="0 0 0"
-        rpy="0 0 0" />
-      <geometry>
-        <mesh
-          filename="package://diablo_bot/description/meshes/l_wrist_Link.STL" />
+          filename="package://diablo_bot/meshes/l_wrist_Link.STL" />
+      </geometry>
+      <material
+        name="">
+        <color
+          rgba="0.752941176470588 0.752941176470588 0.752941176470588 1" />
+      </material>
+    </visual>
+    <collision>
+      <origin
+        xyz="0 0 0"
+        rpy="0 0 0" />
+      <geometry>
+        <mesh
+          filename="package://diablo_bot/meshes/l_wrist_Link.STL" />
       </geometry>
     </collision>
@@ -309,19 +304,19 @@
       <geometry>
         <mesh
-          filename="package://diablo_bot/description/meshes/l_mid_base_Link.STL" />
-      </geometry>
-      <material
-        name="">
-        <color
-          rgba="0.752941176470588 0.752941176470588 0.752941176470588 1" />
-      </material>
-    </visual>
-    <collision>
-      <origin
-        xyz="0 0 0"
-        rpy="0 0 0" />
-      <geometry>
-        <mesh
-          filename="package://diablo_bot/description/meshes/l_mid_base_Link.STL" />
+          filename="package://diablo_bot/meshes/l_mid_base_Link.STL" />
+      </geometry>
+      <material
+        name="">
+        <color
+          rgba="0.752941176470588 0.752941176470588 0.752941176470588 1" />
+      </material>
+    </visual>
+    <collision>
+      <origin
+        xyz="0 0 0"
+        rpy="0 0 0" />
+      <geometry>
+        <mesh
+          filename="package://diablo_bot/meshes/l_mid_base_Link.STL" />
       </geometry>
     </collision>
@@ -367,19 +362,19 @@
       <geometry>
         <mesh
-          filename="package://diablo_bot/description/meshes/l_mid_middle_Link.STL" />
-      </geometry>
-      <material
-        name="">
-        <color
-          rgba="0.752941176470588 0.752941176470588 0.752941176470588 1" />
-      </material>
-    </visual>
-    <collision>
-      <origin
-        xyz="0 0 0"
-        rpy="0 0 0" />
-      <geometry>
-        <mesh
-          filename="package://diablo_bot/description/meshes/l_mid_middle_Link.STL" />
+          filename="package://diablo_bot/meshes/l_mid_middle_Link.STL" />
+      </geometry>
+      <material
+        name="">
+        <color
+          rgba="0.752941176470588 0.752941176470588 0.752941176470588 1" />
+      </material>
+    </visual>
+    <collision>
+      <origin
+        xyz="0 0 0"
+        rpy="0 0 0" />
+      <geometry>
+        <mesh
+          filename="package://diablo_bot/meshes/l_mid_middle_Link.STL" />
       </geometry>
     </collision>
@@ -425,19 +420,19 @@
       <geometry>
         <mesh
-          filename="package://diablo_bot/description/meshes/l_mid_tip_Link.STL" />
-      </geometry>
-      <material
-        name="">
-        <color
-          rgba="0.752941176470588 0.752941176470588 0.752941176470588 1" />
-      </material>
-    </visual>
-    <collision>
-      <origin
-        xyz="0 0 0"
-        rpy="0 0 0" />
-      <geometry>
-        <mesh
-          filename="package://diablo_bot/description/meshes/l_mid_tip_Link.STL" />
+          filename="package://diablo_bot/meshes/l_mid_tip_Link.STL" />
+      </geometry>
+      <material
+        name="">
+        <color
+          rgba="0.752941176470588 0.752941176470588 0.752941176470588 1" />
+      </material>
+    </visual>
+    <collision>
+      <origin
+        xyz="0 0 0"
+        rpy="0 0 0" />
+      <geometry>
+        <mesh
+          filename="package://diablo_bot/meshes/l_mid_tip_Link.STL" />
       </geometry>
     </collision>
@@ -483,19 +478,19 @@
       <geometry>
         <mesh
-          filename="package://diablo_bot/description/meshes/l_thumb_base_Link.STL" />
-      </geometry>
-      <material
-        name="">
-        <color
-          rgba="0.752941176470588 0.752941176470588 0.752941176470588 1" />
-      </material>
-    </visual>
-    <collision>
-      <origin
-        xyz="0 0 0"
-        rpy="0 0 0" />
-      <geometry>
-        <mesh
-          filename="package://diablo_bot/description/meshes/l_thumb_base_Link.STL" />
+          filename="package://diablo_bot/meshes/l_thumb_base_Link.STL" />
+      </geometry>
+      <material
+        name="">
+        <color
+          rgba="0.752941176470588 0.752941176470588 0.752941176470588 1" />
+      </material>
+    </visual>
+    <collision>
+      <origin
+        xyz="0 0 0"
+        rpy="0 0 0" />
+      <geometry>
+        <mesh
+          filename="package://diablo_bot/meshes/l_thumb_base_Link.STL" />
       </geometry>
     </collision>
@@ -541,19 +536,19 @@
       <geometry>
         <mesh
-          filename="package://diablo_bot/description/meshes/l_thumb_middle_Link.STL" />
-      </geometry>
-      <material
-        name="">
-        <color
-          rgba="0.752941176470588 0.752941176470588 0.752941176470588 1" />
-      </material>
-    </visual>
-    <collision>
-      <origin
-        xyz="0 0 0"
-        rpy="0 0 0" />
-      <geometry>
-        <mesh
-          filename="package://diablo_bot/description/meshes/l_thumb_middle_Link.STL" />
+          filename="package://diablo_bot/meshes/l_thumb_middle_Link.STL" />
+      </geometry>
+      <material
+        name="">
+        <color
+          rgba="0.752941176470588 0.752941176470588 0.752941176470588 1" />
+      </material>
+    </visual>
+    <collision>
+      <origin
+        xyz="0 0 0"
+        rpy="0 0 0" />
+      <geometry>
+        <mesh
+          filename="package://diablo_bot/meshes/l_thumb_middle_Link.STL" />
       </geometry>
     </collision>
@@ -599,19 +594,19 @@
       <geometry>
         <mesh
-          filename="package://diablo_bot/description/meshes/l_thumb_tip_Link.STL" />
-      </geometry>
-      <material
-        name="">
-        <color
-          rgba="0.752941176470588 0.752941176470588 0.752941176470588 1" />
-      </material>
-    </visual>
-    <collision>
-      <origin
-        xyz="0 0 0"
-        rpy="0 0 0" />
-      <geometry>
-        <mesh
-          filename="package://diablo_bot/description/meshes/l_thumb_tip_Link.STL" />
+          filename="package://diablo_bot/meshes/l_thumb_tip_Link.STL" />
+      </geometry>
+      <material
+        name="">
+        <color
+          rgba="0.752941176470588 0.752941176470588 0.752941176470588 1" />
+      </material>
+    </visual>
+    <collision>
+      <origin
+        xyz="0 0 0"
+        rpy="0 0 0" />
+      <geometry>
+        <mesh
+          filename="package://diablo_bot/meshes/l_thumb_tip_Link.STL" />
       </geometry>
     </collision>
@@ -657,19 +652,19 @@
       <geometry>
         <mesh
-          filename="package://diablo_bot/description/meshes/l_index_base_Link.STL" />
-      </geometry>
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
File: description/gazebo_plugin.xacro (robot description, xacro)
@@ -6,25 +6,3 @@
         </plugin>
     </gazebo>
-    <gazebo>
-        <plugin name="p3d_base_controller" filename="libgazebo_ros_p3d.so">
-            <rpy_offsets>0 0 0</rpy_offsets>
-            <xyz_offsets>0 0 0</xyz_offsets>
-            <frame_name>base_footprint</frame_name>
-            <gaussian_noise>0.01</gaussian_noise>
-            <topic_name>gazebo_robot_pose</topic_name>
-            <body_name>dummy_root</body_name>
-            <update_rate>50.0</update_rate>
-            <always_on>true</always_on>
-        </plugin>
-    </gazebo>
-    <gazebo>
-        <plugin name="imu_plugin" filename="libgazebo_ros_imu.so">
-            <always_on>true</always_on>
-            <body_name>dummy_root</body_name>
-            <topic_name>imu</topic_name>
-            <service_name>imu_service</service_name>
-            <gaussian_noise>0.0</gaussian_noise>
-            <update_rate>20.0</update_rate>
-        </plugin>
-    </gazebo>
 </robot>

File: description/robot.urdf.xacro (robot description, xacro)
@@ -2,5 +2,6 @@
 <robot xmlns:xacro="http://www.ros.org/wiki/xacro"  name="diablo_robot">
     <xacro:include filename="diablo_core.xacro" />
-    <!--<xacro:include filename="ros2_control.xacro" />
-    <xacro:include filename="gazebo_plugin.xacro" />-->
+    <xacro:include filename="ros2_control.xacro" />
+    <xacro:include filename="gazebo_plugin.xacro" />
+    <xacro:include filename="imu_sensor.xacro" />
 </robot>

File: description/ros2_control.xacro (robot description, xacro)
@@ -55,5 +55,4 @@
             </state_interface>
             <state_interface name='velocity'/>
-            <state_interface name='effort'/>
         </joint>
         <joint name="r1">
@@ -63,5 +62,4 @@
             </state_interface>
             <state_interface name='velocity'/>
-            <state_interface name='effort'/>
         </joint>
         <joint name="l3">
@@ -71,5 +69,4 @@
             </state_interface>
             <state_interface name='velocity'/>
-            <state_interface name='effort'/>
         </joint>
         <joint name="r3">
@@ -79,23 +76,20 @@
             </state_interface>
             <state_interface name='velocity'/>
-            <state_interface name='effort'/>
         </joint>
         <joint name="r4">
             <command_interface name="velocity">
-                <param name="min">-1.0</param>
-                <param name="max">1.0</param>
+                <param name="min">-10.0</param>
+                <param name="max">10.0</param>
             </command_interface>
             <state_interface name='position'/>
             <state_interface name='velocity'/>
-            <state_interface name='effort'/>
         </joint>
         <joint name="l4">
             <command_interface name="velocity">
-                <param name="min">-1.0</param>
-                <param name="max">1.0</param>
+                <param name="min">-10.0</param>
+                <param name="max">10.0</param>
             </command_interface>
             <state_interface name='position'/>
             <state_interface name='velocity'/>
-            <state_interface name='effort'/>
         </joint>
     </ros2_control>
